File: PCB/n8 bus/n8 bus.sch (KiCad schematic (older format))
At the start: 1 part, among them J1 n8 Bus Connector

Commit message: n8 bus card template updated
Connections:
- net USB_D+ is gone; now on net A1: J1.26 (Pin_26)
- net USB_D- is gone; now on net A0: J1.28 (Pin_28)
- net +5V: now also J1.3 (Pin_3), J1.31 (Pin_31), J1.32 (Pin_32), J1.4 (Pin_4); no longer J1.1 (Pin_1), J1.2 (Pin_2), J1.29 (Pin_29), J1.30 (Pin_30)
- net A0: no longer J1.5 (Pin_5)
- net A1: no longer J1.7 (Pin_7)
- net A2: now also J1.24 (Pin_24); no longer J1.9 (Pin_9)
- net A3: now also J1.22 (Pin_22); no longer J1.11 (Pin_11)
- net A4: now also J1.20 (Pin_20); no longer J1.13 (Pin_13)
- net A5: now also J1.18 (Pin_18); no longer J1.15 (Pin_15)
- net CLK: now also J1.12 (Pin_12); no longer J1.21 (Pin_21)
- net D0: now also J1.27 (Pin_27); no longer J1.6 (Pin_6)
- net D1: now also J1.25 (Pin_25); no longer J1.8 (Pin_8)
- net D2: now also J1.23 (Pin_23); no longer J1.10 (Pin_10)
- net D3: now also J1.21 (Pin_21); no longer J1.12 (Pin_12)
- net D4: now also J1.19 (Pin_19); no longer J1.14 (Pin_14)
- net D5: now also J1.17 (Pin_17); no longer J1.16 (Pin_16)
- net D6: now also J1.15 (Pin_15); no longer J1.18 (Pin_18)
- net D7: now also J1.13 (Pin_13); no longer J1.20 (Pin_20)
- net FUTURE0: now also J1.8 (Pin_8); no longer J1.25 (Pin_25)
- net FUTURE1: now also J1.6 (Pin_6); no longer J1.27 (Pin_27)
- net GND: now also J1.1 (Pin_1), J1.2 (Pin_2), J1.29 (Pin_29), J1.30 (Pin_30); no longer J1.3 (Pin_3), J1.31 (Pin_31), J1.32 (Pin_32), J1.4 (Pin_4)
- net R~W: now also J1.14 (Pin_14); no longer J1.19 (Pin_19)
- net ~CS: now also J1.16 (Pin_16); no longer J1.17 (Pin_17)
- net ~IRQ: now also J1.11 (Pin_11); no longer J1.22 (Pin_22)
- net ~NMI: now also J1.9 (Pin_9); no longer J1.24 (Pin_24)
- net ~RES: now also J1.10 (Pin_10); no longer J1.23 (Pin_23)
- new net ~READ: J1.7 (Pin_7)
- new net ~WRITE: J1.5 (Pin_5)
Changed lines of the file:
@@
 L power:+5V #PWR0101
 U 1 1 604C9E8F
-P 925 3000
-F 0 "#PWR0101" H 925 2850 50  0001 C CNN
-F 1 "+5V" H 800 3050 50  0000 C CNN
-F 2 "" H 925 3000 50  0001 C CNN
-F 3 "" H 925 3000 50  0001 C CNN
-	1    925  3000
+P 2100 3000
+F 0 "#PWR0101" H 2100 2850 50  0001 C CNN
+F 1 "+5V" H 1975 3050 50  0000 C CNN
+F 2 "" H 2100 3000 50  0001 C CNN
+F 3 "" H 2100 3000 50  0001 C CNN
+	1    2100 3000
 	1    0    0    -1
 $EndComp
@@
 L power:GND #PWR0102
 U 1 1 604CA2D6
+P 2100 4500
+F 0 "#PWR0102" H 2100 4250 50  0001 C CNN
+F 1 "GND" H 2200 4500 50  0000 C CNN
+F 2 "" H 2100 4500 50  0001 C CNN
+F 3 "" H 2100 4500 50  0001 C CNN
+	1    2100 4500
+	1    0    0    -1
+$EndComp
+Connection ~ 1275 3000
+Wire Wire Line
+	1275 3000 1775 3000
+Wire Wire Line
+	950  4500 1175 4500
+Connection ~ 1275 4500
+Wire Wire Line
+	1275 4500 1775 4500
+$Comp
+L power:+5V #PWR0103
+U 1 1 604CB07B
 P 950 4500
-F 0 "#PWR0102" H 950 4250 50  0001 C CNN
-F 1 "GND" H 800 4450 50  0000 C CNN
+F 0 "#PWR0103" H 950 4350 50  0001 C CNN
+F 1 "+5V" H 1075 4550 50  0000 C CNN
 F 2 "" H 950 4500 50  0001 C CNN
 F 3 "" H 950 4500 50  0001 C CNN
@@
 	1    0    0    -1
 $EndComp
-Connection ~ 1275 3000
-Wire Wire Line
-	1275 3000 1775 3000
-Wire Wire Line
-	950  4500 1175 4500
-Connection ~ 1275 4500
-Wire Wire Line
-	1275 4500 1775 4500
-$Comp
-L power:+5V #PWR0103
-U 1 1 604CB07B
-P 2100 4500
-F 0 "#PWR0103" H 2100 4350 50  0001 C CNN
-F 1 "+5V" H 2225 4550 50  0000 C CNN
-F 2 "" H 2100 4500 50  0001 C CNN
-F 3 "" H 2100 4500 50  0001 C CNN
-	1    2100 4500
-	1    0    0    -1
-$EndComp
 $Comp
 L power:GND #PWR0104
 U 1 1 604CB0E8
-P 2100 3000
-F 0 "#PWR0104" H 2100 2750 50  0001 C CNN
-F 1 "GND" H 2250 2950 50  0000 C CNN
-F 2 "" H 2100 3000 50  0001 C CNN
-F 3 "" H 2100 3000 50  0001 C CNN
-	1    2100 3000
+P 950 2850
+F 0 "#PWR0104" H 950 2600 50  0001 C CNN
+F 1 "GND" H 775 2800 50  0000 C CNN
+F 2 "" H 950 2850 50  0001 C CNN
+F 3 "" H 950 2850 50  0001 C CNN
+	1    950  2850
 	1    0    0    -1
 $EndComp
@@
 	1850 4500 1975 4500
 Entry Wire Line
-	1975 3200 2075 3300
-Entry Wire Line
-	1975 3300 2075 3400
-Entry Wire Line
-	1975 3400 2075 3500
-Entry Wire Line
-	1975 3500 2075 3600
-Entry Wire Line
-	1975 3600 2075 3700
-Entry Wire Line
-	1975 3700 2075 3800
-Entry Wire Line
-	1975 3800 2075 3900
-Entry Wire Line
-	1975 3900 2075 4000
-Wire Wire Line
-	1775 3200 1975 3200
-Wire Wire Line
-	1775 3300 1975 3300
-Wire Wire Line
-	1775 3400 1975 3400
-Wire Wire Line
-	1775 3500 1975 3500
-Wire Wire Line
-	1775 3600 1975 3600
-Wire Wire Line
-	1775 3700 1975 3700
-Wire Wire Line
-	1775 3800 1975 3800
-Wire Wire Line
-	1775 3900 1975 3900
-Text Label 1800 3200 0    50   ~ 0
+	1075 4300 975  4200
+Entry Wire Line
+	1075 4200 975  4100
+Entry Wire Line
+	1075 4100 975  4000
+Entry Wire Line
+	1075 4000 975  3900
+Entry Wire Line
+	1075 3900 975  3800
+Entry Wire Line
+	1075 3800 975  3700
+Entry Wire Line
+	1075 3700 975  3600
+Entry Wire Line
+	1075 3600 975  3500
+Wire Wire Line
+	1275 4300 1075 4300
+Wire Wire Line
+	1275 4200 1075 4200
+Wire Wire Line
+	1275 4100 1075 4100
+Wire Wire Line
+	1275 4000 1075 4000
+Wire Wire Line
+	1275 3900 1075 3900
+Wire Wire Line
+	1275 3800 1075 3800
+Wire Wire Line
+	1275 3700 1075 3700
+Wire Wire Line
+	1275 3600 1075 3600
+Text Label 1250 4300 2    50   ~ 0
 D0
-Text Label 1800 3300 0    50   ~ 0
+Text Label 1250 4200 2    50   ~ 0
 D1
-Text Label 1800 3400 0    50   ~ 0
+Text Label 1250 4100 2    50   ~ 0
 D2
-Text Label 1800 3500 0    50   ~ 0
+Text Label 1250 4000 2    50   ~ 0
 D3
-Text Label 1800 3600 0    50   ~ 0
+Text Label 1250 3900 2    50   ~ 0
 D4
-Text Label 1800 3700 0    50   ~ 0
+Text Label 1250 3800 2    50   ~ 0
 D5
-Text Label 1800 3800 0    50   ~ 0
+Text Label 1250 3700 2    50   ~ 0
 D6
-Text Label 1800 3900 0    50   ~ 0
+Text Label 1250 3600 2    50   ~ 0
 D7
 Entry Wire Line
-	925  3100 1025 3200
-Entry Wire Line
-	925  3200 1025 3300
-Entry Wire Line
-	925  3300 1025 3400
-Entry Wire Line
-	925  3400 1025 3500
-Entry Wire Line
-	925  3500 1025 3600
-Entry Wire Line
-	925  3600 1025 3700
-Wire Wire Line
-	1275 3200 1025 3200
-Wire Wire Line
-	1275 3300 1025 3300
-Wire Wire Line
-	1275 3400 1025 3400
-Wire Wire Line
-	1275 3500 1025 3500
-Wire Wire Line
-	1275 3600 1025 3600
-Wire Wire Line
-	1275 3700 1025 3700
-Text Label 1125 3200 0    50   ~ 0
+	2125 4400 2025 4300
+Entry Wire Line
+	2125 4300 2025 4200
+Entry Wire Line
+	2125 4200 2025 4100
+Entry Wire Line
+	2125 4100 2025 4000
+Entry Wire Line
+	2125 4000 2025 3900
+Entry Wire Line
+	2125 3900 2025 3800
+Wire Wire Line
+	1775 4300 2025 4300
+Wire Wire Line
+	1775 4200 2025 4200
+Wire Wire Line
+	1775 4100 2025 4100
+Wire Wire Line
+	1775 4000 2025 4000
+Wire Wire Line
+	1775 3900 2025 3900
+Wire Wire Line
+	1775 3800 2025 3800
+Text Label 1925 4300 2    50   ~ 0
 A0
-Text Label 1125 3300 0    50   ~ 0
+Text Label 1925 4200 2    50   ~ 0
 A1
-Text Label 1125 3400 0    50   ~ 0
+Text Label 1925 4100 2    50   ~ 0
 A2
-Text Label 1125 3500 0    50   ~ 0
+Text Label 1925 4000 2    50   ~ 0
 A3
-Text Label 1125 3600 0    50   ~ 0
+Text Label 1925 3900 2    50   ~ 0
 A4
-Text Label 1125 3700 0    50   ~ 0
+Text Label 1925 3800 2    50   ~ 0
 A5
-Text GLabel 950  3750 0    50   Input ~ 0
-~CS
-Text GLabel 950  3900 0    50   Input ~ 0
-R~W
-Text GLabel 950  4025 0    50   Input ~ 0
-CLK
-Wire Wire Line
-	1275 3800 1225 3800
-Wire Wire Line
-	1225 3800 1225 3750
-Wire Wire Line
-	1225 3750 950  3750
-Wire Wire Line
-	1275 3900 950  3900
-Wire Wire Line
-	1275 4000 1225 4000
-Wire Wire Line
-	1225 4000 1225 4025
-Wire Wire Line
-	1225 4025 950  4025
-Text GLabel 950  4150 0    50   Input ~ 0
-~RES
-Wire Wire Line
-	1275 4100 1175 4100
-Wire Wire Line
-	1175 4100 1175 4150
-Wire Wire Line
-	1175 4150 950  4150
-Text GLabel 1150 4275 0    50   BiDi ~ 0
-FUTURE0
-Text GLabel 1150 4375 0    50   BiDi ~ 0
-FUTURE1
-Wire Wire Line
-	1275 4200 1150 4200
-Wire Wire Line
-	1150 4200 1150 4275
-Wire Wire Line
-	1275 4300 1200 4300
-Wire Wire Line
-	1200 4300 1200 4375
-Wire Wire Line
-	1200 4375 1150 4375
-Text GLabel 1925 4300 2    50   BiDi ~ 0
-USB_D-
-Text GLabel 1925 4200 2    50   BiDi ~ 0
-USB_D+
-Wire Wire Line
-	1775 4200 1925 4200
-Wire Wire Line
-	1775 4300 1925 4300
-Text GLabel 2125 4075 2    50   Output ~ 0
+Text GLabel 1100 3075 0    50   Output ~ 0
+~WRITE
+Text GLabel 1100 3225 0    50   Output ~ 0
+~READ
+Wire Wire Line
+	1275 3300 1125 3300
+Wire Wire Line
+	1275 3200 1125 3200
+Text GLabel 1100 3375 0    50   Output ~ 0
 ~NMI
-Wire Wire Line
-	1775 4100 2075 4100
-Wire Wire Line
-	2075 4100 2075 4075
-Wire Wire Line
-	2075 4075 2125 4075
-Wire Wire Line
-	1775 4000 1850 4000
-Text GLabel 1850 4000 2    50   Output ~ 0
+Text GLabel 900  3475 0    50   Output ~ 0
 ~IRQ
 $Comp
@@
 	1850 3000 2100 3000
 Wire Wire Line
-	925  3000 1275 3000
+	1050 3000 1275 3000
+Wire Wire Line
+	1050 3000 1050 2850
+Wire Wire Line
+	1050 2850 950  2850
+Wire Wire Line
+	1850 3125 1900 3125
+Wire Wire Line
+	1850 3200 1850 3125
+Wire Wire Line
+	1775 3200 1850 3200
+Wire Wire Line
+	1900 3300 1900 3225
+Wire Wire Line
+	1775 3300 1900 3300
+Text GLabel 1900 3125 2    50   BiDi ~ 0
+FUTURE1
+Text GLabel 1900 3225 2    50   BiDi ~ 0
+FUTURE0
+Wire Wire Line
+	1875 3350 2100 3350
+Wire Wire Line
+	1875 3400 1875 3350
+Wire Wire Line
+	1775 3400 1875 3400
+Text GLabel 2100 3350 2    50   Input ~ 0
+~RES
+Wire Wire Line
+	1825 3475 2100 3475
+Wire Wire Line
+	1825 3500 1825 3475
+Wire Wire Line
+	1775 3500 1825 3500
+Wire Wire Line
+	1775 3600 2100 3600
+Wire Wire Line
+	2025 3700 2025 3750
+Text GLabel 2100 3475 2    50   Input ~ 0
+CLK
+Text GLabel 2100 3600 2    50   Input ~ 0
+R~W
+Text GLabel 2100 3750 2    50   Input ~ 0
+~CS
+Wire Wire Line
+	1775 3700 2025 3700
+Wire Wire Line
+	2025 3750 2100 3750
+Wire Wire Line
+	1125 3200 1125 3075
+Wire Wire Line
+	1125 3075 1100 3075
+Wire Wire Line
+	1125 3300 1125 3225
+Wire Wire Line
+	1125 3225 1100 3225
+Wire Wire Line
+	1275 3500 1050 3500
+Wire Wire Line
+	1050 3500 1050 3475
+Wire Wire Line
+	1050 3475 900  3475
+Wire Wire Line
+	1275 3400 1200 3400
+Wire Wire Line
+	1200 3400 1200 3375
+Wire Wire Line
+	1200 3375 1100 3375
 Wire Bus Line
-	925  3100 925  3600
+	975  3500 975  4200
 Wire Bus Line
-	2075 3300 2075 4000
+	2125 3900 2125 4400
 $EndSCHEMATC
