File: PCB/viaduct/viaduct.sch (KiCad schematic (older format))
At the start: 8 parts, among them J1 n8 Bus, J2 Conn_01x03_Male, J3 Conn_01x03_Male, J4 Conn_02x12, U1 65C22S

Commit message: New placement and parts for v2
Parts:
- J2: value Conn_01x03_Male -> PORT_A_PULLUP_DOWN
- J3: value Conn_01x03_Male -> PORT_B_PULLUP_DOWN
- J4: value Conn_02x12 -> GPIO
Connections:
- no-connect marks 9 -> 7
Other:
- moved on the sheet: J4
Changed lines of the file:
@@
 P 6825 1950
 F 0 "J2" H 6797 1882 50  0000 R CNN
-F 1 "Conn_01x03_Male" H 6797 1973 50  0000 R CNN
+F 1 "PORT_A_PULLUP_DOWN" H 6797 1973 50  0000 R CNN
 F 2 "Connector_PinHeader_2.54mm:PinHeader_1x03_P2.54mm_Vertical" H 6825 1950 50  0001 C CNN
 F 3 "~" H 6825 1950 50  0001 C CNN
@@
 P 6825 3125
 F 0 "J3" H 6797 3057 50  0000 R CNN
-F 1 "Conn_01x03_Male" H 6797 3148 50  0000 R CNN
+F 1 "PORT_B_PULLUP_DOWN" H 6797 3148 50  0000 R CNN
 F 2 "Connector_PinHeader_2.54mm:PinHeader_1x03_P2.54mm_Vertical" H 6825 3125 50  0001 C CNN
 F 3 "~" H 6825 3125 50  0001 C CNN
@@
 L Connector_Generic:Conn_02x12_Odd_Even J4
 U 1 1 6064F493
-P 8275 2750
-F 0 "J4" H 8325 3367 50  0000 C CNN
-F 1 "Conn_02x12" H 8325 2050 50  0000 C CNN
-F 2 "Connector_PinSocket_2.54mm:PinSocket_2x12_P2.54mm_Horizontal" H 8275 2750 50  0001 C CNN
-F 3 "~" H 8275 2750 50  0001 C CNN
-	1    8275 2750
-	1    0    0    -1
-$EndComp
-Entry Wire Line
-	7725 2250 7825 2350
-Entry Wire Line
-	7725 2350 7825 2450
-Entry Wire Line
-	7725 2450 7825 2550
-Entry Wire Line
-	7725 2550 7825 2650
-Entry Wire Line
-	7725 2650 7825 2750
-Entry Wire Line
-	7725 2750 7825 2850
-Entry Wire Line
-	7725 2850 7825 2950
-Entry Wire Line
-	7725 2950 7825 3050
-Wire Wire Line
-	7825 2350 8075 2350
-Wire Wire Line
-	7825 2450 8075 2450
-Wire Wire Line
-	7825 2550 8075 2550
-Wire Wire Line
-	7825 2650 8075 2650
-Wire Wire Line
-	7825 2750 8075 2750
-Wire Wire Line
-	7825 2850 8075 2850
-Wire Wire Line
-	7825 2950 8075 2950
-Wire Wire Line
-	7825 3050 8075 3050
-Text Label 8000 2350 2    50   ~ 0
+P 8550 2750
+F 0 "J4" H 8600 3425 50  0000 C CNN
+F 1 "GPIO" H 8600 3350 50  0000 C CNN
+F 2 "Connector_PinSocket_2.54mm:PinSocket_2x12_P2.54mm_Horizontal" H 8550 2750 50  0001 C CNN
+F 3 "~" H 8550 2750 50  0001 C CNN
+	1    8550 2750
+	1    0    0    -1
+$EndComp
+Entry Wire Line
+	8000 2250 8100 2350
+Entry Wire Line
+	8000 2350 8100 2450
+Entry Wire Line
+	8000 2450 8100 2550
+Entry Wire Line
+	8000 2550 8100 2650
+Entry Wire Line
+	8000 2650 8100 2750
+Entry Wire Line
+	8000 2750 8100 2850
+Entry Wire Line
+	8000 2850 8100 2950
+Entry Wire Line
+	8000 2950 8100 3050
+Wire Wire Line
+	8100 2350 8350 2350
+Wire Wire Line
+	8100 2450 8350 2450
+Wire Wire Line
+	8100 2550 8350 2550
+Wire Wire Line
+	8100 2650 8350 2650
+Wire Wire Line
+	8100 2750 8350 2750
+Wire Wire Line
+	8100 2850 8350 2850
+Wire Wire Line
+	8100 2950 8350 2950
+Wire Wire Line
+	8100 3050 8350 3050
+Text Label 8275 2350 2    50   ~ 0
 PA0
-Text Label 8000 2450 2    50   ~ 0
+Text Label 8275 2450 2    50   ~ 0
 PA1
-Text Label 8000 2550 2    50   ~ 0
+Text Label 8275 2550 2    50   ~ 0
 PA2
-Text Label 8000 2650 2    50   ~ 0
+Text Label 8275 2650 2    50   ~ 0
 PA3
-Text Label 8000 2750 2    50   ~ 0
+Text Label 8275 2750 2    50   ~ 0
 PA4
-Text Label 8000 2850 2    50   ~ 0
+Text Label 8275 2850 2    50   ~ 0
 PA5
-Text Label 8000 2950 2    50   ~ 0
+Text Label 8275 2950 2    50   ~ 0
 PA6
-Text Label 8000 3050 2    50   ~ 0
+Text Label 8275 3050 2    50   ~ 0
 PA7
 Text GLabel 5025 1825 2    50   BiDi ~ 0
@@
 Wire Wire Line
 	3675 3725 3825 3725
-Text GLabel 7975 3150 0    50   BiDi ~ 0
+Text GLabel 8250 3150 0    50   BiDi ~ 0
 CA1
-Text GLabel 7975 3250 0    50   BiDi ~ 0
+Text GLabel 8250 3250 0    50   BiDi ~ 0
 CA2
 Wire Wire Line
-	7975 3150 8075 3150
-Wire Wire Line
-	7975 3250 8075 3250
-Wire Wire Line
-	8575 2350 8825 2350
-Wire Wire Line
-	8575 2450 8825 2450
-Wire Wire Line
-	8575 2550 8825 2550
-Wire Wire Line
-	8575 2650 8825 2650
-Wire Wire Line
-	8575 2750 8825 2750
-Wire Wire Line
-	8575 2850 8825 2850
-Wire Wire Line
-	8575 2950 8825 2950
-Wire Wire Line
-	8575 3050 8825 3050
-Text Label 8600 2350 0    50   ~ 0
+	8250 3150 8350 3150
+Wire Wire Line
+	8250 3250 8350 3250
+Wire Wire Line
+	8850 2350 9100 2350
+Wire Wire Line
+	8850 2450 9100 2450
+Wire Wire Line
+	8850 2550 9100 2550
+Wire Wire Line
+	8850 2650 9100 2650
+Wire Wire Line
+	8850 2750 9100 2750
+Wire Wire Line
+	8850 2850 9100 2850
+Wire Wire Line
+	8850 2950 9100 2950
+Wire Wire Line
+	8850 3050 9100 3050
+Text Label 8875 2350 0    50   ~ 0
 PB0
-Text Label 8600 2450 0    50   ~ 0
+Text Label 8875 2450 0    50   ~ 0
 PB1
-Text Label 8600 2550 0    50   ~ 0
+Text Label 8875 2550 0    50   ~ 0
 PB2
-Text Label 8600 2650 0    50   ~ 0
+Text Label 8875 2650 0    50   ~ 0
 PB3
-Text Label 8600 2750 0    50   ~ 0
+Text Label 8875 2750 0    50   ~ 0
 PB4
-Text Label 8600 2850 0    50   ~ 0
+Text Label 8875 2850 0    50   ~ 0
 PB5
-Text Label 8600 2950 0    50   ~ 0
+Text Label 8875 2950 0    50   ~ 0
 PB6
-Text Label 8600 3050 0    50   ~ 0
+Text Label 8875 3050 0    50   ~ 0
 PB7
-Text GLabel 8675 3250 2    50   BiDi ~ 0
+Text GLabel 8950 3250 2    50   BiDi ~ 0
 CB2
-Text GLabel 8675 3150 2    50   BiDi ~ 0
+Text GLabel 8950 3150 2    50   BiDi ~ 0
 CB1
 Wire Wire Line
-	8575 3150 8675 3150
-Wire Wire Line
-	8575 3250 8675 3250
-Entry Wire Line
-	8925 2350 8825 2450
-Entry Wire Line
-	8925 2250 8825 2350
-Entry Wire Line
-	8925 2450 8825 2550
-Entry Wire Line
-	8925 2550 8825 2650
-Entry Wire Line
-	8925 2650 8825 2750
-Entry Wire Line
-	8925 2750 8825 2850
-Entry Wire Line
-	8925 2850 8825 2950
-Entry Wire Line
-	8925 2950 8825 3050
+	8850 3150 8950 3150
+Wire Wire Line
+	8850 3250 8950 3250
+Entry Wire Line
+	9200 2350 9100 2450
+Entry Wire Line
+	9200 2250 9100 2350
+Entry Wire Line
+	9200 2450 9100 2550
+Entry Wire Line
+	9200 2550 9100 2650
+Entry Wire Line
+	9200 2650 9100 2750
+Entry Wire Line
+	9200 2750 9100 2850
+Entry Wire Line
+	9200 2850 9100 2950
+Entry Wire Line
+	9200 2950 9100 3050
 $Comp
 L Device:C_Small C1
@@
 Wire Wire Line
 	2675 2125 2850 2125
-NoConn ~ 2400 3600
-NoConn ~ 1900 3600
-$Comp
-L power:+5V #PWR?
-U 1 1 612D5945
-P 8000 2250
-F 0 "#PWR?" H 8000 2100 50  0001 C CNN
-F 1 "+5V" H 8015 2423 50  0000 C CNN
-F 2 "" H 8000 2250 50  0001 C CNN
-F 3 "" H 8000 2250 50  0001 C CNN
-	1    8000 2250
-	1    0    0    -1
-$EndComp
-$Comp
-L power:GND #PWR?
-U 1 1 612D63AA
-P 8000 3350
-F 0 "#PWR?" H 8000 3100 50  0001 C CNN
-F 1 "GND" H 8005 3177 50  0000 C CNN
-F 2 "" H 8000 3350 50  0001 C CNN
-F 3 "" H 8000 3350 50  0001 C CNN
-	1    8000 3350
-	1    0    0    -1
-$EndComp
-Wire Wire Line
-	8000 2250 8075 2250
-Wire Wire Line
-	8075 2250 8575 2250
-Connection ~ 8075 2250
-Wire Wire Line
-	8000 3350 8075 3350
-Wire Wire Line
-	8075 3350 8575 3350
+$Comp
+L power:+5V #PWR0106
+U 1 1 605A3179
+P 8250 2250
+F 0 "#PWR0106" H 8250 2100 50  0001 C CNN
+F 1 "+5V" H 8265 2423 50  0000 C CNN
+F 2 "" H 8250 2250 50  0001 C CNN
+F 3 "" H 8250 2250 50  0001 C CNN
+	1    8250 2250
+	1    0    0    -1
+$EndComp
+Wire Wire Line
+	8350 2250 8250 2250
+Wire Wire Line
+	8350 2250 8850 2250
+Connection ~ 8350 2250
+$Comp
+L power:GND #PWR0112
+U 1 1 605B293E
+P 8250 3350
+F 0 "#PWR0112" H 8250 3100 50  0001 C CNN
+F 1 "GND" H 8255 3177 50  0000 C CNN
+F 2 "" H 8250 3350 50  0001 C CNN
+F 3 "" H 8250 3350 50  0001 C CNN
+	1    8250 3350
+	1    0    0    -1
+$EndComp
+Wire Wire Line
+	8350 3350 8250 3350
+Wire Wire Line
+	8350 3350 8850 3350
+Connection ~ 8350 3350
 Wire Bus Line
 	5125 2025 5125 2325
@@
 	5700 3025 5700 3725
 Wire Bus Line
-	7725 2250 7725 2950
-Wire Bus Line
-	8925 2250 8925 2950
-Connection ~ 8075 3350
+	8000 2250 8000 2950
+Wire Bus Line
+	9200 2250 9200 2950
 $EndSCHEMATC

Commit message: release candidate for v2
Parts:
- J1: value n8 Bus -> n8 Bus Connector
- U1: symbol 6502:65C22S -> viaduct-rescue:65C22S-6502
- renumbered J4 to J2, J2 to J3, J3 to J4
Connections:
- net +5V: now also J1.3 (Pin_3), J1.31 (Pin_31), J1.32 (Pin_32), J1.4 (Pin_4); no longer J1.1 (Pin_1), J1.2 (Pin_2)
- net CLK: now also J1.12 (Pin_12); no longer J1.21 (Pin_21)
- net D0: now also J1.27 (Pin_27); no longer J1.6 (Pin_6)
- net D1: now also J1.25 (Pin_25); no longer J1.8 (Pin_8)
- net D2: now also J1.23 (Pin_23); no longer J1.10 (Pin_10)
- net D3: now also J1.21 (Pin_21); no longer J1.12 (Pin_12)
- net D4: now also J1.19 (Pin_19); no longer J1.14 (Pin_14)
- net D5: now also J1.17 (Pin_17); no longer J1.16 (Pin_16)
- net D6: now also J1.15 (Pin_15); no longer J1.18 (Pin_18)
- net D7: now also J1.13 (Pin_13); no longer J1.20 (Pin_20)
- net GND: now also J1.1 (Pin_1), J1.2 (Pin_2), J1.29 (Pin_29), J1.30 (Pin_30); no longer J1.3 (Pin_3), J1.31 (Pin_31), J1.32 (Pin_32), J1.4 (Pin_4)
- net RS0: now also J1.28 (Pin_28); no longer J1.5 (Pin_5)
- net RS1: now also J1.26 (Pin_26); no longer J1.7 (Pin_7)
- net RS2: now also J1.24 (Pin_24); no longer J1.9 (Pin_9)
- net RS3: now also J1.22 (Pin_22); no longer J1.11 (Pin_11)
- net R~W: now also J1.14 (Pin_14); no longer J1.19 (Pin_19)
- net ~CS: now also J1.16 (Pin_16); no longer J1.17 (Pin_17)
- net ~IRQ: now also J1.11 (Pin_11); no longer J1.22 (Pin_22)
- net ~RES: now also J1.10 (Pin_10); no longer J1.23 (Pin_23)
- no-connect marks 7 -> 5
