File: PCB/kids serial/kids serial.sch (KiCad schematic (older format))
At the start: 6 parts, among them J1 n8 Bus Connector, J2 UARTConnector, J3 PowerViaUSB, U1 6551, X1 CXO_DIP14

Commit message: New placement and parts for v2
Parts:
- removed J2: UARTConnector, Connector_PinSocket_2.54mm:PinSocket_1x06_P2.54mm_Horizontal, symbol Connector_Generic:Conn_01x06
- removed J3: PowerViaUSB, Connector_PinHeader_2.54mm:PinHeader_1x02_P2.54mm_Vertical, symbol Connector_Generic:Conn_01x02
- removed U1: 6551, Package_DIP:DIP-28_W15.24mm_Socket, symbol 65xx:6551
- added C2, C3: 100nF, Capacitor_THT:C_Disc_D5.0mm_W2.5mm_P2.50mm, symbol Device:C_Small
- added C4, C5: 47pF, Capacitor_THT:C_Disc_D3.8mm_W2.6mm_P2.50mm, symbol Device:C_Small
- added D1: TX, LED_THT:LED_D3.0mm, symbol Device:LED
- added D2: RX, LED_THT:LED_D3.0mm, symbol Device:LED
- added R1, R2: 330, Resistor_THT:R_Axial_DIN0207_L6.3mm_D2.5mm_P7.62mm_Horizontal, symbol Device:R
- added R3, R4: 27, Resistor_THT:R_Axial_DIN0207_L6.3mm_D2.5mm_P7.62mm_Horizontal, symbol Device:R
- added U1: SC28L92_PLC44, Package_LCC:PLCC-44_THT-Socket, symbol 65xx:SC28L92_PLC44
- added U2: FT230XS, Package_SO:SSOP-16_3.9x4.9mm_P0.635mm, symbol Interface_USB:FT230XS
- C1: value 100nf -> 100nF
- X1: value CXO_DIP14 -> 3.6864Mhz; footprint Oscillator:Oscillator_DIP-14 -> Oscillator:Oscillator_DIP-8; symbol Oscillator:CXO_DIP14 -> Oscillator:CXO_DIP8
Connections:
- net +5V: now also X1.8 (Vcc), C2.1, U1.44 (VCC), U2.12 (VCC); no longer X1.14 (Vcc)
- net A0: now also U1.2 (A0)
- net A1: now also U1.4 (A1)
- net A2: now also U1.6 (A2)
- net A3: now also U1.7 (A3)
- net D0: now also U1.28 (D0)
- net D1: now also U1.18 (D1)
- net D2: now also U1.27 (D2)
- net D3: now also U1.19 (D3)
- net D4: now also U1.26 (D4)
- net D5: now also U1.20 (D5)
- net D6: now also U1.25 (D6)
- net D7: now also U1.21 (D7)
- net GND: now also X1.4 (GND), C2.2, C3.2, C4.2, C5.2, U1.12 (I/M), U1.22 (GND), U2.13 (GND), U2.5 (GND); no longer X1.7 (GND)
- net R~W: now also U1.9 (~WRN)
- net XTAL_CLK: now also X1.5 (OUT), U1.36 (X1/CLK); no longer X1.8 (OUT)
- net ~CS: now also U1.39 (~CEN)
- net ~IRQ: now also U1.24 (~INTRN)
- net ~RES: now also U1.38 (RESET)
- net USB_D+: now reaches J1.26 (Pin_26)
- net USB_D+: now also C5.1, R4.2
- net USB_D-: now reaches J1.28 (Pin_28)
- net USB_D-: now also C4.1, R3.2
- net CLK: no longer names the net of J1.21 (Pin_21)
- new net: D2.1 (K), U2.14 (CBUS1)
- new net: D1.1 (K), U2.15 (CBUS0)
- new net: R4.1, U2.8 (USBDP)
- new net: R3.1, U2.9 (USBDM)
- new net: D1.2 (A), R1.2
- new net: D2.2 (A), R2.2
- new net +3V3: C3.1, R1.1, R2.1, U2.10 (3V3OUT), U2.11 (~RESET), U2.3 (VCCIO)
- new net RxD: U1.35 (RxDA), U2.1 (TXD)
- new net TxD: U1.33 (TxDA), U2.4 (RXD)
- new net ~CTS: U1.8 (IP0), U2.2 (~RTS)
- new net ~RTS: U1.32 (OP0), U2.6 (~CTS)
- no-connect marks 13 -> 26
Other:
- note added: "Configured for \n68xxx Bus Mode"

Commit message: v2 changes
Parts:
- removed C2, C3: 100nF, Capacitor_THT:C_Disc_D5.0mm_W2.5mm_P2.50mm, symbol Device:C_Small
- removed C4, C5: 47pF, Capacitor_THT:C_Disc_D3.8mm_W2.6mm_P2.50mm, symbol Device:C_Small
- removed D1: TX, LED_THT:LED_D3.0mm, symbol Device:LED
- removed D2: RX, LED_THT:LED_D3.0mm, symbol Device:LED
- removed R1, R2: 330, Resistor_THT:R_Axial_DIN0207_L6.3mm_D2.5mm_P7.62mm_Horizontal, symbol Device:R
- removed R3, R4: 27, Resistor_THT:R_Axial_DIN0207_L6.3mm_D2.5mm_P7.62mm_Horizontal, symbol Device:R
- removed U1: SC28L92_PLC44, Package_LCC:PLCC-44_THT-Socket, symbol 65xx:SC28L92_PLC44
- removed U2: FT230XS, Package_SO:SSOP-16_3.9x4.9mm_P0.635mm, symbol Interface_USB:FT230XS
- added J2: UARTConnector, Connector_PinSocket_2.54mm:PinSocket_1x06_P2.54mm_Horizontal, symbol Connector_Generic:Conn_01x06
- added J3: PowerViaUSB, Connector_PinHeader_2.54mm:PinHeader_1x02_P2.54mm_Vertical, symbol Connector_Generic:Conn_01x02
- added U1: 6551, Package_DIP:DIP-28_W15.24mm_Socket, symbol 65xx:6551
- C1: value 100nF -> 100nf
- X1: value 3.6864Mhz -> CXO_DIP14; footprint Oscillator:Oscillator_DIP-8 -> Oscillator:Oscillator_DIP-14; symbol Oscillator:CXO_DIP8 -> Oscillator:CXO_DIP14
Connections:
- net USB_D+ is gone; now on net A1: J1.26 (Pin_26)
- net USB_D- is gone; now on net A0: J1.28 (Pin_28)
- net +5V: now also J1.3 (Pin_3), J1.31 (Pin_31), J1.32 (Pin_32), J1.4 (Pin_4), X1.14 (Vcc), J3.1 (Pin_1), U1.15 (VCC), U1.2 (CS1); no longer J1.1 (Pin_1), J1.2 (Pin_2), J1.29 (Pin_29), J1.30 (Pin_30), X1.8 (Vcc)
- net A0: now also U1.13 (RS0); no longer J1.5 (Pin_5)
- net A1: now also U1.14 (RS1); no longer J1.7 (Pin_7)
- net A2: now also J1.24 (Pin_24); no longer J1.9 (Pin_9)
- net A3: now also J1.22 (Pin_22); no longer J1.11 (Pin_11)
- net A4: now also J1.20 (Pin_20); no longer J1.13 (Pin_13)
- net A5: now also J1.18 (Pin_18); no longer J1.15 (Pin_15)
- net D0: now also J1.27 (Pin_27), U1.18 (D0); no longer J1.6 (Pin_6)
- net D1: now also J1.25 (Pin_25), U1.19 (D1); no longer J1.8 (Pin_8)
- net D2: now also J1.23 (Pin_23), U1.20 (D2); no longer J1.10 (Pin_10)
- net D3: now also J1.21 (Pin_21), U1.21 (D3); no longer J1.12 (Pin_12)
- net D4: now also J1.19 (Pin_19), U1.22 (D4); no longer J1.14 (Pin_14)
- net D5: now also J1.17 (Pin_17), U1.23 (D5); no longer J1.16 (Pin_16)
- net D6: now also J1.15 (Pin_15), U1.24 (D6); no longer J1.18 (Pin_18)
- net D7: now also J1.13 (Pin_13), U1.25 (D7); no longer J1.20 (Pin_20)
- net GND: now also J1.1 (Pin_1), J1.2 (Pin_2), J1.29 (Pin_29), J1.30 (Pin_30), X1.7 (GND), J2.2 (Pin_2), U1.1 (VSS), U1.16 (~DCD), U1.17 (~DSR); no longer J1.3 (Pin_3), J1.31 (Pin_31), J1.32 (Pin_32), J1.4 (Pin_4), X1.4 (GND)
- net R~W: now also J1.14 (Pin_14), U1.28 (R/~W); no longer J1.19 (Pin_19)
- net XTAL_CLK: now also X1.8 (OUT), U1.6 (XTAL1); no longer X1.5 (OUT)
- net ~CS: now also J1.16 (Pin_16), U1.3 (~CS2); no longer J1.17 (Pin_17)
- net ~IRQ: now also J1.11 (Pin_11), U1.26 (~IRQ); no longer J1.22 (Pin_22)
- net ~RES: now also J1.10 (Pin_10), U1.4 (~RES); no longer J1.23 (Pin_23)
- new net CLK: J1.12 (Pin_12), U1.27 (ϕ2)
- new net RXD_IO: J2.4 (Pin_4), U1.10 (TxD)
- new net TXD_IO: J2.3 (Pin_3), U1.12 (RxD)
- new net VCC_IO: J2.1 (Pin_1), J3.2 (Pin_2)
- new net ~CTS_IO: J2.6 (Pin_6), U1.8 (~RTS)
- new net ~RTS_IO: J2.5 (Pin_5), U1.9 (~CTS)
- no-connect marks 26 -> 9
Other:
- note removed: "Configured for \n68xxx Bus Mode"
