File: PCB/n8 bit special/n8 bit special.sch (KiCad schematic (older format))
At the start: 35 parts, among them J1 PowerPort, J2 PORT0, J3 PORT2, J4 PORT1, J5 PORT3, J6 Conn_02x08_Odd_Even, SW1 SW_Push_Dual, U1 W65C02SxP, U2 CY62256-70PC, U3 CY62256-70PC, U4 28C256, U5 74LS21, U6 22V10C, U7 DS1813, X1 2Mhz

Commit message: New placement and parts for v2
Parts:
- removed C10: 100nf, Capacitor_THT:C_Disc_D5.0mm_W2.5mm_P2.50mm, symbol Device:C_Small
- removed J1: PowerPort, Connector_PinSocket_2.54mm:PinSocket_1x04_P2.54mm_Vertical, symbol Connector_Generic:Conn_01x04
- removed J5: PORT3, Connector_PinSocket_2.54mm:PinSocket_2x16_P2.54mm_Vertical, symbol Connector_Generic:Conn_02x16_Odd_Even
- removed R3: 3K3, Resistor_THT:R_Axial_DIN0207_L6.3mm_D2.5mm_P7.62mm_Horizontal, symbol Device:R
- added C16: 100nf, Capacitor_THT:C_Disc_D5.0mm_W2.5mm_P2.50mm, symbol Device:C_Small
- added C17, C18: 100nF, Capacitor_THT:C_Disc_D5.0mm_W2.5mm_P2.50mm, symbol Device:C_Small
- added C19, C20: 47pF, Capacitor_THT:C_Disc_D5.0mm_W2.5mm_P2.50mm, symbol Device:C_Small
- added D2: TX, LED_THT:LED_D3.0mm, symbol Device:LED
- added D3: RX, LED_THT:LED_D3.0mm, symbol Device:LED
- added J1: USB_B_Micro, Connector_USB:USB_Micro-B_Amphenol_10118194_Horizontal, symbol Connector:USB_B_Micro
- added Q1: 2N3904, Package_TO_SOT_THT:TO-92, symbol Transistor_BJT:2N3904
- added R4: 10K, Resistor_THT:R_Axial_DIN0207_L6.3mm_D2.5mm_P7.62mm_Horizontal, symbol Device:R
- added R5, R6: 220, Resistor_THT:R_Axial_DIN0207_L6.3mm_D2.5mm_P7.62mm_Horizontal, symbol Device:R
- added R7, R8: 27, Resistor_THT:R_Axial_DIN0207_L6.3mm_D2.5mm_P7.62mm_Horizontal, symbol Device:R
- added U10: 74HC00, Package_DIP:DIP-14_W7.62mm_Socket, symbol 74xx:74HC00
- added U8: SC28L92_PLC44, Package_LCC:PLCC-44_THT-Socket, symbol 65xx:SC28L92_PLC44
- added U9: FT230XS, Package_SO:SSOP-16_3.9x4.9mm_P0.635mm, symbol Interface_USB:FT230XS
- C2: value 1000uF -> 470uF; footprint Capacitor_THT:CP_Radial_D10.0mm_P5.00mm -> Capacitor_THT:CP_Radial_D8.0mm_P3.80mm
- C9: value 100nf -> 100nF
- J6: footprint Connector_PinHeader_2.54mm:PinHeader_2x08_P2.54mm_Vertical -> Connector_PinHeader_2.54mm:PinHeader_2x06_P2.54mm_Vertical; symbol Connector_Generic:Conn_02x08_Odd_Even -> Connector_Generic:Conn_02x06_Odd_Even
- R1: value 330 -> 220
- U1: footprint Package_DIP:DIP-40_W15.24mm_Socket -> Package_LCC:PLCC-44_THT-Socket; symbol 65xx:W65C02SxP -> 65xx:W65C02SxPL
- X1: value 2Mhz -> 3.6864Mhz; footprint Oscillator:Oscillator_DIP-14 -> Oscillator:Oscillator_DIP-8; symbol Oscillator:CXO_DIP14 -> Oscillator:CXO_DIP8
- renumbered C7 to C5, C8 to C6, C5 to C7, C6 to C8
Connections:
- net +5V: now also C9.1, U1.37 (VDD), U1.42 (~SO), U1.9 (VDD), U5.13, X1.8 (Vcc), C16.2, C17.1, J1.1 (VBUS), Q1.3 (C), U10.14 (VCC), U8.12 (I/M), U8.44 (VCC), U9.12 (VCC); no longer C9.2, U1.38 (~SO), U1.8 (VDD), X1.14 (Vcc)
- net A0: now also U1.10 (A0), U8.2 (A0); no longer U1.9 (A0)
- net A1: now also U1.11 (A1), U8.4 (A1); no longer U1.10 (A1)
- net A10: now also U1.21 (A10); no longer U1.19 (A10)
- net A11: now also U1.22 (A11); no longer U1.20 (A11)
- net A12: now also U1.25 (A12); no longer U1.22 (A12)
- net A13: now also U1.26 (A13); no longer U1.23 (A13)
- net A14: now also U1.27 (A14); no longer U1.24 (A14)
- net A15: now also U1.28 (A15); no longer U1.25 (A15)
- net A2: now also U1.13 (A2), U8.6 (A2); no longer U1.11 (A2)
- net A3: now also U1.14 (A3), U8.7 (A3); no longer U1.12 (A3)
- net A4: now also U1.15 (A4); no longer U1.13 (A4)
- net A5: now also U1.16 (A5); no longer U1.14 (A5)
- net A6: now also U1.17 (A6); no longer U1.15 (A6)
- net A7: now also U1.18 (A7); no longer U1.16 (A7)
- net A8: now also U1.19 (A8); no longer U1.17 (A8)
- net A9: now also U1.20 (A9); no longer U1.18 (A9)
- net CLK: now also U1.41 (ϕ0), X1.5 (OUT), U10.2, U10.4, U8.36 (X1/CLK); no longer U1.37 (ϕ0), X1.8 (OUT)
- net D0: now also U1.36 (D0), U8.28 (D0); no longer U1.33 (D0)
- net D1: now also U1.35 (D1), U8.18 (D1); no longer U1.32 (D1)
- net D2: now also U1.34 (D2), U8.27 (D2); no longer U1.31 (D2)
- net D3: now also U1.33 (D3), U8.19 (D3); no longer U1.30 (D3)
- net D4: now also U1.32 (D4), U8.26 (D4); no longer U1.29 (D4)
- net D5: now also U1.31 (D5), U8.20 (D5); no longer U1.28 (D5)
- net D6: now also U1.30 (D6), U8.25 (D6); no longer U1.27 (D6)
- net D7: now also U1.29 (D7), U8.21 (D7); no longer U1.26 (D7)
- net FUTURE0: now also U6.15 (IO14); no longer U6.16 (IO15)
- net FUTURE1: now also U6.14 (IO13); no longer U6.15 (IO14)
- net GND: now also C9.2, U1.1 (VSS), U1.23 (VSS), U1.24 (VSS), X1.4 (GND), C16.1, C17.2, C18.2, C19.2, C20.2, J1.5 (GND), U10.7 (GND), U8.22 (GND), U9.13 (GND), U9.5 (GND); no longer C9.1, U1.21 (VSS), U2.22 (~OE), U3.22 (~OE), U4.22 (~OE), X1.7 (GND)
- net R~W: now also U1.38 (R/~W), U10.10, U10.5, U10.9; no longer U1.34 (R/~W), U2.27 (~WE), U3.27 (~WE)
- net USB_D+: now also C20.1, J1.3 (D+), R8.2; no longer J2.26 (Pin_26), J3.26 (Pin_26), J4.26 (Pin_26)
- net USB_D-: now also C19.1, J1.2 (D-), R7.2; no longer J2.28 (Pin_28), J3.28 (Pin_28), J4.28 (Pin_28)
- net ~IRQ: now also U1.5 (~IRQ); no longer U1.4 (~IRQ)
- net ~NMI: now also U1.7 (~NMI); no longer U1.6 (~NMI)
- net ~RES: now also U1.44 (~RES), R4.2, U10.12, U10.13; no longer D1.2 (A), U1.40 (~RES)
- net at U1.2 (~VP): no longer R2.1
- net RDY_PULLUP: now reaches U1.3 (RDY)
- net RDY_PULLUP: now also RN1.2 (R1)
- net at J6.2 (Pin_2): now also RN1.4 (R3); no longer RN1.2 (R1)
- net at J6.4 (Pin_4): now also RN1.5 (R4); no longer RN1.3 (R2)
- net at J6.6 (Pin_6): now also RN1.6 (R5); no longer RN1.4 (R3)
- net at J6.8 (Pin_8): now also RN1.7 (R6); no longer RN1.5 (R4)
- net at J6.10 (Pin_10): now also RN1.8 (R7); no longer RN1.6 (R5)
- net at J6.12 (Pin_12): now also RN1.9 (R8); no longer RN1.7 (R6)
- net PORT3_IRQ_PULLUP renamed ~UART_IRQ
- net ~UART_IRQ: now also R2.1, U8.24 (~INTRN); no longer J6.13 (Pin_13)
- removed net PORT3_NMI_PULLUP: J6.15 (Pin_15), U5.13
- net ~PORT3_CS renamed ~UART_CS
- net ~UART_CS: now also U8.39 (~CEN)
- new net: D1.2 (A), Q1.1 (E)
- new net: Q1.2 (B), R4.1
- new net: U10.1, U10.8
- new net: D3.1 (K), U9.14 (CBUS1)
- new net: D2.1 (K), U9.15 (CBUS0)
- new net: R8.1, U9.8 (USBDP)
- new net: R7.1, U9.9 (USBDM)
- new net: D2.2 (A), R5.2
- new net: D3.2 (A), R6.2
- new net +3V3: C18.1, R5.1, R6.1, U9.10 (3V3OUT), U9.11 (~RESET), U9.3 (VCCIO)
- new net BE_PULLUP: RN1.3 (R2), U1.40 (BE)
- new net RxD: U8.35 (RxDA), U9.1 (TXD)
- new net TxD: U8.33 (TxDA), U9.4 (RXD)
- new net UART_RES: U10.11, U8.38 (RESET)
- new net ~CTS: U8.8 (IP0), U9.2 (~RTS)
- new net ~READ: J2.26 (Pin_26), J3.26 (Pin_26), J4.26 (Pin_26), U10.6, U2.22 (~OE), U3.22 (~OE), U4.22 (~OE), U8.10 (~RDN)
- new net ~RTS: U8.32 (OP0), U9.6 (~CTS)
- new net ~WRITE: J2.28 (Pin_28), J3.28 (Pin_28), J4.28 (Pin_28), U10.3, U2.27 (~WE), U3.27 (~WE), U8.9 (~WRN)
- no-connect marks 7 -> 27
Other:
- note added: "Clock Qualified Read/Write"
- note added: "Configured for \nIntel Bus Mode"
- note added: "UART and USB"
- moved on the sheet: C2, D1, R1, RN1, X1

Commit message: Layout centered around USB D+/D- differential pair
Connections:
- net at U9.15 (CBUS0): no longer D2.1 (K)
- net at U9.7 (CBUS2): now also D2.1 (K)
- net F_USB_D+: now reaches R8.1, U9.8 (USBDP)
- net F_USB_D-: now reaches R7.1, U9.9 (USBDM)
- no-connect marks 27 -> 28
Other:
- moved on the sheet: C9, D2, D3, R5, R6, U10A, U10B, U10C, U10E

Commit message: Cleanup
Other:
- note added: "Qualified Signals"
- note removed: "Clock Qualified Read/Write"
- moved on the sheet: C9, U10D, U10E
Changed lines of the file:
@@
 L 74xx:74HC00 U10
 U 4 1 61A96A90
-P 13075 6850
-F 0 "U10" H 13075 7175 50  0000 C CNN
-F 1 "74HC00" H 13075 7084 50  0000 C CNN
-F 2 "Package_DIP:DIP-14_W7.62mm_Socket" H 13075 6850 50  0001 C CNN
-F 3 "http://www.ti.com/lit/gpn/sn74hc00" H 13075 6850 50  0001 C CNN
-	4    13075 6850
+P 12300 5050
+F 0 "U10" H 12300 5375 50  0000 C CNN
+F 1 "74HC00" H 12300 5284 50  0000 C CNN
+F 2 "Package_DIP:DIP-14_W7.62mm_Socket" H 12300 5050 50  0001 C CNN
+F 3 "http://www.ti.com/lit/gpn/sn74hc00" H 12300 5050 50  0001 C CNN
+	4    12300 5050
 	1    0    0    -1
 $EndComp
@@
 L 74xx:74HC00 U10
 U 5 1 61A99ED9
-P 12025 5025
-F 0 "U10" H 12255 5071 50  0000 L CNN
-F 1 "74HC00" H 12255 4980 50  0000 L CNN
-F 2 "Package_DIP:DIP-14_W7.62mm_Socket" H 12025 5025 50  0001 C CNN
-F 3 "http://www.ti.com/lit/gpn/sn74hc00" H 12025 5025 50  0001 C CNN
-	5    12025 5025
+P 14100 5050
+F 0 "U10" H 14330 5096 50  0000 L CNN
+F 1 "74HC00" H 14330 5005 50  0000 L CNN
+F 2 "Package_DIP:DIP-14_W7.62mm_Socket" H 14100 5050 50  0001 C CNN
+F 3 "http://www.ti.com/lit/gpn/sn74hc00" H 14100 5050 50  0001 C CNN
+	5    14100 5050
 	1    0    0    -1
 $EndComp
@@
 	8975 4200 8975 5875
 Text Notes 9000 4150 0    50   ~ 0
-Clock Qualified Read/Write
-Wire Notes Line
-	12775 5875 12775 4200
-Wire Notes Line
-	8975 5875 12775 5875
-Wire Notes Line
-	8975 4200 12775 4200
+Qualified Signals
+Wire Notes Line
+	14750 5875 14750 4200
+Wire Notes Line
+	8975 5875 14750 5875
+Wire Notes Line
+	8975 4200 14750 4200
 $Comp
 L power:GND #PWR0125
 U 1 1 62A886B4
-P 12025 5575
-F 0 "#PWR0125" H 12025 5325 50  0001 C CNN
-F 1 "GND" H 12025 5400 50  0000 C CNN
-F 2 "" H 12025 5575 50  0001 C CNN
-F 3 "" H 12025 5575 50  0001 C CNN
-	1    12025 5575
-	1    0    0    -1
-$EndComp
-Wire Wire Line
-	12025 5525 12025 5550
+P 14100 5600
+F 0 "#PWR0125" H 14100 5350 50  0001 C CNN
+F 1 "GND" H 14100 5425 50  0000 C CNN
+F 2 "" H 14100 5600 50  0001 C CNN
+F 3 "" H 14100 5600 50  0001 C CNN
+	1    14100 5600
+	1    0    0    -1
+$EndComp
+Wire Wire Line
+	14100 5550 14100 5575
 $Comp
 L power:+5V #PWR0137
 U 1 1 62AF287A
-P 12025 4450
-F 0 "#PWR0137" H 12025 4300 50  0001 C CNN
-F 1 "+5V" H 12040 4623 50  0000 C CNN
-F 2 "" H 12025 4450 50  0001 C CNN
-F 3 "" H 12025 4450 50  0001 C CNN
-	1    12025 4450
-	1    0    0    -1
-$EndComp
-Wire Wire Line
-	12025 4525 12025 4500
-Wire Wire Line
-	12775 6750 12675 6750
-Wire Wire Line
-	12675 6750 12675 6850
-Wire Wire Line
-	12675 6950 12775 6950
-Text GLabel 12575 6850 0    50   Input ~ 0
+P 14100 4475
+F 0 "#PWR0137" H 14100 4325 50  0001 C CNN
+F 1 "+5V" H 14115 4648 50  0000 C CNN
+F 2 "" H 14100 4475 50  0001 C CNN
+F 3 "" H 14100 4475 50  0001 C CNN
+	1    14100 4475
+	1    0    0    -1
+$EndComp
+Wire Wire Line
+	14100 4550 14100 4525
+Wire Wire Line
+	12000 4950 11900 4950
+Wire Wire Line
+	11900 4950 11900 5050
+Wire Wire Line
+	11900 5150 12000 5150
+Text GLabel 11800 5050 0    50   Input ~ 0
 ~RES
 Wire Wire Line
-	12575 6850 12675 6850
-Connection ~ 12675 6850
-Wire Wire Line
-	12675 6850 12675 6950
-Text GLabel 13450 6850 2    50   Output ~ 0
+	11800 5050 11900 5050
+Connection ~ 11900 5050
+Wire Wire Line
+	11900 5050 11900 5150
+Text GLabel 12675 5050 2    50   Output ~ 0
 UART_RES
 Wire Wire Line
-	13375 6850 13450 6850
+	12600 5050 12675 5050
 Text GLabel 11400 8950 2    50   Input ~ 0
 ~WRITE
@@
 L Device:C_Small C9
 U 1 1 63B30DBA
-P 11675 5075
-F 0 "C9" H 11500 5125 50  0000 L CNN
-F 1 "100nF" H 11275 5025 50  0000 L CNN
-F 2 "Capacitor_THT:C_Disc_D5.0mm_W2.5mm_P2.50mm" H 11675 5075 50  0001 C CNN
-F 3 "~" H 11675 5075 50  0001 C CNN
-	1    11675 5075
-	1    0    0    -1
-$EndComp
-Wire Wire Line
-	12025 4500 11675 4500
-Wire Wire Line
-	11675 4500 11675 4975
-Connection ~ 12025 4500
-Wire Wire Line
-	12025 4500 12025 4450
-Wire Wire Line
-	11675 5175 11675 5550
-Wire Wire Line
-	11675 5550 12025 5550
-Connection ~ 12025 5550
-Wire Wire Line
-	12025 5550 12025 5575
+P 13750 5100
+F 0 "C9" H 13575 5150 50  0000 L CNN
+F 1 "100nF" H 13350 5050 50  0000 L CNN
+F 2 "Capacitor_THT:C_Disc_D5.0mm_W2.5mm_P2.50mm" H 13750 5100 50  0001 C CNN
+F 3 "~" H 13750 5100 50  0001 C CNN
+	1    13750 5100
+	1    0    0    -1
+$EndComp
+Wire Wire Line
+	14100 4525 13750 4525
+Wire Wire Line
+	13750 4525 13750 5000
+Connection ~ 14100 4525
+Wire Wire Line
+	14100 4525 14100 4475
+Wire Wire Line
+	13750 5200 13750 5575
+Wire Wire Line
+	13750 5575 14100 5575
+Connection ~ 14100 5575
+Wire Wire Line
+	14100 5575 14100 5600
 NoConn ~ 4450 4200
 NoConn ~ 14925 8250
@@
 Wire Wire Line
 	14925 8450 15675 8450
-Wire Bus Line
-	9800 6675 9800 6975
-Wire Bus Line
-	3475 8975 3475 9475
-Wire Bus Line
-	6375 6250 6375 6750
-Wire Bus Line
-	3475 6250 3475 6750
-Wire Bus Line
-	10300 1450 10300 2150
-Wire Bus Line
-	7700 3225 7700 3925
-Wire Bus Line
-	4475 6250 4475 6950
-Wire Bus Line
-	12775 1450 12775 2150
-Wire Bus Line
-	7375 6250 7375 6950
-Wire Bus Line
-	4475 8975 4475 9675
-Wire Bus Line
-	15025 1425 15025 2125
-Wire Bus Line
-	9800 7225 9800 7925
-Wire Bus Line
-	3225 3400 3225 4300
-Wire Bus Line
-	8700 1450 8700 2850
-Wire Bus Line
-	7700 1525 7700 3025
-Wire Bus Line
-	11175 1450 11175 2850
-Wire Bus Line
-	13625 1425 13625 2825
 $Comp
 L Interface_USB:FT230XS U9
@@
 Text Label 13500 8150 0    50   ~ 0
 F_USB_D+
+Wire Bus Line
+	9800 6675 9800 6975
+Wire Bus Line
+	3475 8975 3475 9475
+Wire Bus Line
+	6375 6250 6375 6750
+Wire Bus Line
+	3475 6250 3475 6750
+Wire Bus Line
+	10300 1450 10300 2150
+Wire Bus Line
+	7700 3225 7700 3925
+Wire Bus Line
+	4475 6250 4475 6950
+Wire Bus Line
+	12775 1450 12775 2150
+Wire Bus Line
+	7375 6250 7375 6950
+Wire Bus Line
+	4475 8975 4475 9675
+Wire Bus Line
+	15025 1425 15025 2125
+Wire Bus Line
+	9800 7225 9800 7925
+Wire Bus Line
+	3225 3400 3225 4300
+Wire Bus Line
+	8700 1450 8700 2850
+Wire Bus Line
+	7700 1525 7700 3025
+Wire Bus Line
+	11175 1450 11175 2850
+Wire Bus Line
+	13625 1425 13625 2825
 $EndSCHEMATC

Commit message: v2 changes
Parts:
- U9: footprint Package_SO:SSOP-16_3.9x4.9mm_P0.635mm -> graphics:SSOP-16_3.9x4.9mm_P0.635mm_long_pads
Changed lines of the file:
@@
 F 0 "U9" H 13850 8850 50  0000 C CNN
 F 1 "FT230XS" H 13850 8775 50  0000 C CNN
-F 2 "Package_SO:SSOP-16_3.9x4.9mm_P0.635mm" H 15225 7550 50  0001 C CNN
+F 2 "graphics:SSOP-16_3.9x4.9mm_P0.635mm_long_pads" H 15225 7550 50  0001 C CNN
 F 3 "https://www.ftdichip.com/Support/Documents/DataSheets/ICs/DS_FT230X.pdf" H 14225 8150 50  0001 C CNN
 	1    14225 8150
