File: PCB/PixelJuice_OpAmpStage/PixelJuice_OpAmpStage.kicad_sch (KiCad schematic)
At the start: 27 parts, among them U5 4066, U6 LM1881, U7 AD8054

Commit message: added 2 new soundcard designs
Parts:
- removed C13, C14, C15: 47uF, Capacitor_THT:CP_Radial_D4.0mm_P2.00mm, symbol Device:C_Polarized_Small
- removed C16: 10nF, Capacitor_SMD:C_0805_2012Metric_Pad1.18x1.45mm_HandSolder, symbol Device:C_Small
- removed R13: 1K, Resistor_SMD:R_0805_2012Metric_Pad1.20x1.40mm_HandSolder, symbol Device:R_Small
- removed R8, R9: 1k, Resistor_SMD:R_0805_2012Metric_Pad1.20x1.40mm_HandSolder, symbol Device:R_Small
- removed U5: 4066, Package_DIP:DIP-14_W7.62mm_Socket, symbol 4xxx:4066
- removed unit 4 of U7
- added C3: 100nF, Capacitor_SMD:C_0805_2012Metric_Pad1.18x1.45mm_HandSolder, symbol Device:C_Small
- added C7, C8, C9: 100nf, Capacitor_SMD:C_0805_2012Metric_Pad1.18x1.45mm_HandSolder, symbol Device:C_Small
- added R11, R12: 680R, Resistor_SMD:R_0805_2012Metric_Pad1.20x1.40mm_HandSolder, symbol Device:R_Small
- added U1: CD4053B, Package_DIP:DIP-16_W7.62mm_Socket, symbol Analog_Switch:CD4053B
- added unit 4 of U3
- added U5: THS7314, Package_SO:SOIC-8_3.9x4.9mm_P1.27mm, symbol VDP:THS7314
- C1: renamed from C8; footprint (none) -> Capacitor_SMD:C_0805_2012Metric_Pad1.18x1.45mm_HandSolder
- J1, J2: renamed from J?; footprint (none) -> Connector_PinHeader_2.54mm:PinHeader_1x05_P2.54mm_Vertical
- R1: value 680k -> 560K
- R2: value 10k -> 910R
- R3: value 10k -> 160R
- R4: value 2k -> 680R
- R5: value 2k -> 620R
- R6: value 2k -> 910R
- R7: value 1k -> 910R
- renumbered C9 to C2, C10 to C4, C11 to C5, C12 to C6, R11 to R10, R12 to R8, R10 to R9, U6 to U2, U7 to U3
Connections:
- net +5V: now also C3.1, R11.1, U1.16 (VDD), U5.4 (VCC)
- net B-Y: now also U1.13 (A1)
- net B-Y_{out}: now also R10.2
- net GND: now also R5.1, R6.1, R7.1, C3.2, R12.1, U1.6 (INH), U1.7 (VEE), U1.8 (VSS), U5.5 (GND)
- net R-Y: now also U1.3 (C1)
- net R-Y_{out}: now also R8.2
- net Y: now also U1.1 (B1), U1.2 (B0); no longer C1.1, U3.3 (+)
- net Y_{out}: now also R9.2
- net ~{BURST}: now also U1.10 (S2), U1.11 (S1), U1.9 (S3)
- net at U3.9 (-): now also R2.1, U3.8; no longer R6.2
- net at R8.1: now also U5.8; no longer U3.8
- net at R3.1: now also U3.1, U3.2 (-); no longer U3.10 (+)
- net at U3.5 (+): now also U1.14 (A); no longer R2.1
- net at R5.2: now also R2.2, C7.1; no longer U3.6 (-)
- net at R10.1: now also U5.6; no longer U3.7
- removed net VREF: R2.2, R3.2, R4.1, R5.1, R6.1
- new net: U1.4 (C), U3.10 (+)
- new net: R9.1, U5.7
- new net: R11.2, R12.2, U3.12 (+)
- new net: U3.13 (-), U3.14
- new net: U1.15 (B), U3.3 (+)
- new net: C7.2, U5.1 (Ch1)
- new net: C8.2, U5.2 (Ch2)
- new net: C9.2, U5.3 (Ch3)
- new net: C9.1, R4.2, R7.2
- new net: R4.1, U3.6 (-), U3.7
- new net SAMPLE: U1.12 (A0), U1.5 (C0)
- new net Y_{DIV}: C1.1, C8.1, R3.2, R6.2
Other:
- note added: "Unused?"
- note removed: "Vref Detector"
- moved on the sheet: C1, C2, C4, C5, C6, J2, R1, R10, R8, R9, U2, U3A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
