File: PCB/bouncer/bouncer.kicad_sch (KiCad schematic)
At the start: 15 parts, among them J1 Conn_01x08_Female, SW1 SW_Push_Dual, SW2 SW_Push_Dual, SW3 SW_Push_Dual, U1 74HC14

Commit message: added 2 new soundcard designs
Parts:
- C1, C2, C4: footprint Capacitor_THT:CP_Radial_D5.0mm_P2.50mm -> Capacitor_THT:CP_Radial_D4.0mm_P2.00mm
- J1: footprint Connector_PinHeader_2.54mm:PinHeader_1x08_P2.54mm_Vertical -> Connector_PinSocket_2.54mm:PinSocket_1x08_P2.54mm_Vertical

Commit message: rc1 for SPI Gate (prev SPI master) rc1 for Bouncer
Parts:
- added H1, H2, H3, H4: MountingHole, MountingHole:MountingHole_3.2mm_M3_DIN965_Pad, symbol Mechanical:MountingHole
Connections:
- no-connect marks 6 -> 0
Other:
- moved on the sheet: C1, C2, C3, C4, J1, R1, R2, R3, R5, R6, SW1, SW2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
