File: PCB/Yamahawk1/Yamahawk1.kicad_pcb (KiCad board)
At the start: 2 copper layers, 99.7 x 52.7 mm, 13 parts, among them J1 n8 Bus Connector, J3 Conn_02x08_Odd_Even, U1 YM2149, U5 65C22S

Commit message: Added SpiMaster support
Parts:
- removed C6: 4.7uF, Capacitor_THT:CP_Radial_D6.3mm_P2.50mm
- removed R11: 1K6, Resistor_THT:R_Axial_DIN0207_L6.3mm_D2.5mm_P10.16mm_Horizontal
- added C2: 4.7uF, Capacitor_THT:CP_Radial_D6.3mm_P2.50mm, F.Cu at (133.1, 44.8)
- added C3: 4.7uF, Capacitor_THT:CP_Radial_D6.3mm_P2.50mm, F.Cu at (133.1, 52.7)
- added CON1: SJ1-3523N, Connector_Audio:Jack_3.5mm_CUI_SJ1-3515N_Horizontal, F.Cu at (184.3, 106.1)
- added R1: 3K, Resistor_THT:R_Axial_DIN0207_L6.3mm_D2.5mm_P10.16mm_Horizontal, F.Cu at (118.5, 42.9)
- added R2: 3K, Resistor_THT:R_Axial_DIN0207_L6.3mm_D2.5mm_P10.16mm_Horizontal, F.Cu at (118.5, 47.0)
- added R3: 3K, Resistor_THT:R_Axial_DIN0207_L6.3mm_D2.5mm_P10.16mm_Horizontal, F.Cu at (118.5, 51.0)
- added R4: 1K, Resistor_THT:R_Axial_DIN0207_L6.3mm_D2.5mm_P10.16mm_Horizontal, F.Cu at (118.5, 55.1)
- C5: value 4.7uF -> 220uf
- J3: value Conn_02x08_Odd_Even -> SPKR_{OUT}
- R10: value 1K6 -> 10R
- R5: value 3K -> 1K
- R6, R7: value 3K -> 1K6
- R8, R9: value 1K -> 8K2
Connections:
- C5 pad 1: Net-(C5-Pad1) -> Net-(C4-Pad1)
- C5 pad 2: /LEFT -> Net-(J3-Pin_1)
- J3 pad 1: GND -> Net-(J3-Pin_1)
- J3 pad 10: CS_{SPI} -> (no net)
- J3 pad 11: +5V -> (no net)
- J3 pad 12: +5V -> (no net)
- J3 pad 13: unconnected-(J3-Pin_13-Pad13) -> (no net)
- J3 pad 14: unconnected-(J3-Pin_13-Pad13) -> (no net)
- J3 pad 15: GND -> (no net)
- J3 pad 16: GND -> (no net)
- J3 pad 3: MISO_{SPI} -> (no net)
- J3 pad 4: MISO_{SPI} -> (no net)
- J3 pad 5: CLK_{SPI} -> (no net)
- J3 pad 6: CLK_{SPI} -> (no net)
- J3 pad 7: MOSI_{SPI} -> (no net)
- J3 pad 8: MOSI_{SPI} -> (no net)
- J3 pad 9: CS_{SPI} -> (no net)
- R10 pad 1: Net-(C6-Pad1) -> Net-(C4-Pad2)
- R10 pad 2: CH_C -> GND
- R5 pad 1: CH_C -> Net-(C3-Pad1)
- R5 pad 2: GND -> CH_A
- R6 pad 1: CH_A -> Net-(C3-Pad1)
- R6 pad 2: GND -> CH_C
- R7 pad 1: CH_B -> Net-(C2-Pad1)
- R7 pad 2: GND -> CH_C
- R8 pad 1: Net-(C5-Pad1) -> AMP_{RIGHT}
- R8 pad 2: CH_B -> Net-(U2-+)
- R9 pad 1: Net-(C6-Pad1) -> AMP_{LEFT}
- R9 pad 2: CH_A -> Net-(U2-+)
- U5 pad 10: CS_{SPI} -> unconnected-(U5-PB0-Pad10)
- U5 pad 11: MOSI_{SPI} -> unconnected-(U5-PB1-Pad11)
- U5 pad 12: CLK_{SPI} -> unconnected-(U5-PB2-Pad12)
- U5 pad 17: MISO_{SPI} -> unconnected-(U5-PB7-Pad17)
