File: PCB/Yamahawk1/Yamahawk1.kicad_sch (KiCad schematic)
At the start: 23 parts, among them CON1 SJ1-3523N, J1 n8 Bus Connector, J2 Conn_01x03_Pin, J3 SPKR_{OUT}, J4 Mini-DIN-6, U1 YM2149, U2 LM386, U5 65C22S

Commit message: Added SpiMaster support
Parts:
- CON1: footprint rc2014:Headphone_Jack_3.5mm_5_pin -> Connector_Audio:Jack_3.5mm_CUI_SJ1-3515N_Horizontal
