File: PCB/Yamahawk2/Yamahawk2.kicad_sch (KiCad schematic)
At the start: 19 parts, among them J1 n8 Bus Connector, U1 MCP6022, U2 YMF262, U4 MCP6022, X1 14.31818 MHz

Commit message: Worked on Spi master a little bit
Parts:
- added C10, C9: 68pf, symbol Device:C_Small
- added C11, C13: 2N7, symbol Device:C_Small
- added C12, C14, C15: 10uf, symbol Device:C_Polarized_Small
- added R10, R12, R14: 10k, symbol Device:R_Small
- added R11, R13: 220, symbol Device:R_Small
- added R5, R8, R9: 22K, symbol Device:R_Small
- added R6, R7: 10K, symbol Device:R_Small
- added U5: OP283GS, symbol Amplifier_Operational:OP283GS
- R2: value 10K -> 220
Connections:
- net +5V: now also C5.1, C6.1, C7.1, U3.6 (FSEL), U3.9 (TST1)
- net +5VA: now also R7.2, U5.8 (V+); no longer U3.9 (TST1)
- net CH_{1}: now also C11.1, U5.3 (+)
- net CH_{2}: now also C13.1, U5.5 (+)
- net GND: now also C5.2, C6.2, C7.2, R6.1
- net at C8.2, R3.2, U4.7: now also C12.1
- net at R2.2: now also C14.2, R12.2; no longer U4.5 (+)
- new net: R5.1, R6.2, R7.1
- new net: C15.2, R13.2, R14.2
- new net: C10.2, R5.2
- new net: C12.2, R10.2, R11.2
- new net: C14.1, U5.1, U5.2 (-)
- new net: C15.1, U5.6 (-), U5.7
- new net GNDA: C11.2, C13.2, R12.1, R14.1, U5.4 (V-)
Other:
- moved on the sheet: C1, C2, C3, C4, C5, C6, C7, C8, J1, L1, R1, R3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

Commit message: Added SpiMaster support
Parts:
- removed C10: 68pf, symbol Device:C_Small
- removed C12: 10uf, symbol Device:C_Polarized_Small
- removed C8: 100pf, symbol Device:C_Small
- removed R10: 10k, symbol Device:R_Small
- removed R11: 220, symbol Device:R_Small
- removed R8, R9: 22K, symbol Device:R_Small
- removed U4: MCP6022, symbol Amplifier_Operational:MCP6022
- added C8: 10uf, symbol Device:C_Polarized_Small
- added CON1: SJ1-3523N, Connector_Audio:Jack_3.5mm_CUI_SJ1-3515N_Horizontal, symbol Connector_Audio:AudioJack3_SwitchTR
- added U4: OP283GS, symbol Amplifier_Operational:OP283GS
- C9: value 68pf -> 2N7
- R3: value 22K -> 220
- R4, R5: value 22K -> 10k
- R6: value 10K -> 1K
- R7: value 10K -> 10k
- U2: symbol Yamaha:YMF262 -> Retro:YMF262M
- U3: symbol Yamaha:YAC512 -> Retro:YAC512
Connections:
- net +5VA: no longer R7.2
- net CH_{1}: now also C9.1, R6.2
- net GND: no longer R4.1, R6.1
- net GNDA: now also C9.2, R4.1, R5.1, R7.1
- net at R5.2: now also R6.1, R7.2, U4.3 (+)
- net at R4.2: now also R3.2, C8.2; no longer R3.1
- new net: C8.1, U4.1, U4.2 (-)
